Commit message: Add Lidar, DepthCam, Imu

File: urdf/robot.urdf.xacro (robot description, xacro)
@@ -2,3 +2,6 @@
 <robot xmlns:xacro="http://www.ros.org/wiki/xacro" name="my_robot">
     <xacro:include filename="$(find robot_description)/urdf/robot_core.xacro"/>
+    <xacro:include filename="$(find robot_description)/urdf/lidar.xacro"/>
+    <xacro:include filename="$(find robot_description)/urdf/imu.xacro"/>
+    <xacro:include filename="$(find robot_description)/urdf/depth_camera.xacro"/>
 </robot>

File: urdf/robot_core.xacro (robot description, xacro)
@@ -48,4 +48,13 @@
     </xacro:macro>
     <xacro:property name="caster_xoff" value="0.14"/>
+    <!-- Robot Footprint -->
+    <link name="base_footprint">
+        <xacro:box_inertial m="15" w="${base_width}" d="${base_length}" h="${base_height}"/>
+    </link>
+    <joint name="base_joint" type="fixed">
+        <parent link="base_link"/>
+        <child link="base_footprint"/>
+        <origin xyz="0.0 0.0 -${wheel_radius+wheel_zoff}" rpy="0 0 0"/>
+    </joint>
      <!-- Robot Base -->
     <link name="base_link">
@@ -62,13 +71,9 @@
         </collision>
     </link>
-    <!-- Robot Footprint -->
-    <link name="base_footprint">
-        <xacro:box_inertial m="15" w="${base_width}" d="${base_length}" h="${base_height}"/>
-    </link>
-    <joint name="base_joint" type="fixed">
-        <parent link="base_link"/>
-        <child link="base_footprint"/>
-        <origin xyz="0.0 0.0 -${wheel_radius+wheel_zoff}" rpy="0 0 0"/>
-    </joint>
+    <gazebo reference="base_link">
+        <material>
+            Gazebo/White
+        </material>
+    </gazebo>
     <!-- Wheels -->
     <xacro:macro name="wheel" params="prefix x_reflect y_reflect">
@@ -95,4 +100,9 @@
             <axis xyz="0 1 0"/>
         </joint>
+        <gazebo reference="${prefix}_link">
+            <material>
+                Gazebo/Black
+            </material>
+        </gazebo>
     </xacro:macro>
     <xacro:wheel prefix="drive_left" x_reflect="-1" y_reflect="1" />
@@ -118,3 +128,10 @@
         <origin xyz="${caster_xoff} 0.0 ${-base_height/2}" rpy="0 0 0"/>
     </joint>
+    <gazebo reference="front_caster">
+        <material>
+            Gazebo/Black
+        </material>
+        <mu1>0.001</mu1>
+        <mu2>0.001</mu2>
+    </gazebo>
 </robot>
