Commit message: Update file

File: urdf/lidar.xacro (robot description, xacro)
@@ -2,5 +2,5 @@
 <robot xmlns:xacro="http://www.ros.org/wiki/xacro" name="my_robot">
     <!-- Add Gazebo Lidar Plugin -->
-    <link name="lidar_link">
+    <link name="laser_frame">
         <inertial>
             <origin xyz="0 0 0" rpy="0 0 0"/>
@@ -23,9 +23,10 @@
     <joint name="lidar_joint" type="fixed">
         <parent link="base_link"/>
-        <child link="lidar_link"/>
+        <child link="laser_frame"/>
         <origin xyz="0 0 0.12" rpy="0 0 0"/>
     </joint>
-    <gazebo reference="lidar_link">
-        <sensor name="lidar" type="ray">
+    <gazebo reference="laser_frame">
+        <sensor name="laser" type="ray">\
+            <pose>0 0 0 0 0 0</pose>
             <always_on>true</always_on>
             <visualize>true</visualize>
@@ -57,5 +58,5 @@
                 </ros>
                 <output_type>sensor_msgs/LaserScan</output_type>
-                <frame_name>lidar_link</frame_name>
+                <frame_name>laser_frame</frame_name>
             </plugin>
         </sensor>

File: urdf/robot.urdf.xacro (robot description, xacro)
@@ -5,3 +5,5 @@
     <xacro:include filename="$(find robot_description)/urdf/imu.xacro"/>
     <xacro:include filename="$(find robot_description)/urdf/depth_camera.xacro"/>
+    <xacro:include filename="$(find robot_description)/urdf/gazebo_control.xacro"/>
+    <xacro:include filename="$(find robot_description)/urdf/ros2_control.xacro"/>
 </robot>

File: urdf/robot_core.xacro (robot description, xacro)
@@ -106,6 +106,6 @@
         </gazebo>
     </xacro:macro>
-    <xacro:wheel prefix="drive_left" x_reflect="-1" y_reflect="1" />
-    <xacro:wheel prefix="drive_right" x_reflect="-1" y_reflect="-1" />
+    <xacro:wheel prefix="left_wheel" x_reflect="-1" y_reflect="1" />
+    <xacro:wheel prefix="right_wheel" x_reflect="-1" y_reflect="-1" />
     <!-- Caster Wheel -->
     <link name="front_caster">
