Commit message: Update urdf mecanum

File: urdf/gazebo_control.xacro (robot description, xacro)
@@ -2,10 +2,17 @@
 <robot xmlns:xacro="http://www.ros.org/wiki/xacro">
     <gazebo>
-        <plugin name="diff_drive" filename="libgazebo_ros_diff_drive.so">
+        <plugin name="mecanum_drive_controller" filename="libgazebo_ros_planar_move.so">
+            <ros>
+                <namespace>/</namespace>
+                <remapping>cmd_vel:=cmd_vel</remapping>
+                <remapping>odom:=odom</remapping>
+            </ros>
+            <alwaysOn>true</alwaysOn>
+            <updateRate>100</updateRate>
             <!-- Wheel Information -->
-            <left_joint>left_wheel_joint</left_joint>
-            <right_joint>right_wheel_joint</right_joint>
-            <wheel_separation>0.4</wheel_separation>
-            <wheel_diameter>0.2</wheel_diameter>
+            <front_left_joint>front_left_joint</front_left_joint>
+            <front_right_joint>front_right_joint</front_right_joint>
+            <back_left_joint>back_left_joint</back_left_joint>
+            <back_right_joint>back_right_joint</back_right_joint>
             <!-- Limits -->
             <max_wheel_torque>200</max_wheel_torque>

File: urdf/robot.urdf.xacro (robot description, xacro)
@@ -6,4 +6,4 @@
     <xacro:include filename="$(find robot_description)/urdf/depth_camera.xacro"/>
     <xacro:include filename="$(find robot_description)/urdf/gazebo_control.xacro"/>
-    <xacro:include filename="$(find robot_description)/urdf/ros2_control.xacro"/>
+    <!-- <xacro:include filename="$(find robot_description)/urdf/ros2_control.xacro"/> -->
 </robot>

File: urdf/robot_core.xacro (robot description, xacro)
@@ -101,4 +101,6 @@
         </joint>
         <gazebo reference="${prefix}_link">
+            <mu1>0.1</mu1>
+            <mu2>0.1</mu2>
             <material>
                 Gazebo/Black
@@ -106,8 +108,10 @@
         </gazebo>
     </xacro:macro>
-    <xacro:wheel prefix="left_wheel" x_reflect="-1" y_reflect="1" />
-    <xacro:wheel prefix="right_wheel" x_reflect="-1" y_reflect="-1" />
+    <xacro:wheel prefix="front_left" x_reflect="1" y_reflect="1" />
+    <xacro:wheel prefix="front_right" x_reflect="1" y_reflect="-1" />
+    <xacro:wheel prefix="back_left" x_reflect="-1" y_reflect="1" />
+    <xacro:wheel prefix="back_right" x_reflect="-1" y_reflect="-1" />
     <!-- Caster Wheel -->
-    <link name="front_caster">
+    <!-- <link name="front_caster">
         <visual>
             <geometry>
@@ -134,4 +138,4 @@
         <mu1>0.001</mu1>
         <mu2>0.001</mu2>
-    </gazebo>
+    </gazebo> -->
 </robot>
